File: PCB/DIY-PCB_EAGLE/Esquematico_PCB_DIY_V1.sch (EAGLE design)
At the start: 2 parts

Commit message: PCB_EAGLE CHANGES
Parts:
- added R2, R3, R4, R5, R6: (no value), rcl:R-US_R0805
- added SV1: (no value), con-lstb:MA04-1
- added T1, T2, T3, T4: (no value), zetex:NMOSSOT23
Connections:
- new net N$2: R3.2, T1.G
- new net N$4: R4.2, T2.G
- new net N$5: R5.2, T3.G
- new net N$6: R6.2, T4.G
- net BOOT: now also R2.2, SV1.2
- net GND: now also R2.1, SV1.1, T1.S, T2.S, T3.S, T4.S
- net PWM0: now also R3.1
- net PWM1: now also R4.1
- net PWM2: now also R5.1
- net PWM3: now also R6.1
- net RX: now also SV1.3
- net TX: now also SV1.4
- net VCC: now also T1.D, T2.D, T3.D, T4.D
