File: PCB/DIY-PCB_EAGLE/Esquematico_PCB_DIY_V1.sch (EAGLE design)
At the start: 2 parts

Commit message: Esquematico
Parts:
- added C1: 4u7, rcl:C-USC0805K
- added C10, C3, C6, C7: 0.1uF, rcl:C-USC0805K
- added C11, C5, C8: 10nF, rcl:C-USC0805K
- added C2, C9: 47uF, rcl:C-USC0805K
- added C4: 2.2nF, rcl:C-USC0805K
- added IC1: BMP280, bosch-bmp280:BMP280
- added L1: 4u7, inductor-neosid:MS85
- added R10, R13, R14, R15, R16, R2, R3, R4, R5, R6, R7, R8, R9: (no value), rcl:R-US_R0805
- added R11, R12: 10K, rcl:R-US_R0805
- added R17, R18: 1K, rcl:R-US_R0805
- added SV1: (no value), con-lstb:MA04-1
- added T1, T2, T3, T4: (no value), zetex:NMOSSOT23
- added U$1: MPU-6050, invensense:MPU-6050
- added U$2: LM3671, texas-custom:LM3671
- added X1: 22-23-2021, con-molex:22-23-2021
Connections:
- new net N$10: C3.1, U$1.REGOUT
- new net N$11: C4.1, U$1.CPOUT
- new net N$13: IC1.SDO
- new net N$2: R3.2, T1.G
- new net N$3: L1.1, U$2.SW
- new net N$4: R4.2, T2.G
- new net N$5: R5.2, T3.G
- new net N$6: R6.2, T4.G
- new net N$7: R13.2, R14.1
- new net N$8: R15.1, R16.2, U$1.AD0
- new net VCC_BAT: C1.1, U$2.EN, U$2.VIN
- net ADC: now also R11.1, R12.1
- net BOOT: now also SV1.2
- net GND: now also C1.2, C10.2, C11.2, C2.2, C3.2, C4.2, C5.2, C6.2, C7.2, IC1.GND, R10.1, R12.2, R13.1, R16.1, R2.1, R7.1, R8.1, R9.1, SV1.1, T1.S, T2.S, T3.S, T4.S, U$1.GND, U$2.GND, X1-2.S
- net I2C_SCL: now also IC1.SCK, R18.1, U$1.SCL
- net I2C_SDA: now also IC1.SDI, R17.1, U$1.SDA
- net PWM0: now also R3.1, R7.2
- net PWM1: now also R4.1, R8.2
- net PWM2: now also R10.2, R5.1
- net PWM3: now also R6.1, R9.2
- net RX: now also SV1.3
- net TX: now also SV1.4
- net VCC: now also C10.1, C11.1, C2.1, C5.1, C6.1, C7.1, C8.1, C9.1, IC1.CSB, IC1.VDD, IC1.VDDIO, L1.2, R11.2, R14.2, R15.2, R17.2, R18.2, T1.D, T2.D, T3.D, T4.D, U$1.VDD, U$1.VLOGIC, U$2.FB, X1-1.S
Other:
- moved on the sheet: R1, U1

Commit message: Esquematico
Parts:
- R1, R10, R7, R8, R9: value (none) -> 10K
- R3, R4, R5, R6: value (none) -> 10
Connections:
- new net N$12: U$1.INT
Changed lines of the file:
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@@
 <parts>
 <part name="U1" library="esp8266modules" deviceset="ESP12E" device="SMD"/>
-<part name="R1" library="rcl" deviceset="R-US_" device="R0805"/>
+<part name="R1" library="rcl" deviceset="R-US_" device="R0805" value="10K"/>
 <part name="P+1" library="supply1" deviceset="VCC" device=""/>
 <part name="GND1" library="supply1" deviceset="GND" device=""/>
@@
 <part name="GND6" library="supply1" deviceset="GND" device=""/>
 <part name="GND7" library="supply1" deviceset="GND" device=""/>
-<part name="R3" library="rcl" deviceset="R-US_" device="R0805"/>
-<part name="R4" library="rcl" deviceset="R-US_" device="R0805"/>
-<part name="R5" library="rcl" deviceset="R-US_" device="R0805"/>
-<part name="R6" library="rcl" deviceset="R-US_" device="R0805"/>
+<part name="R3" library="rcl" deviceset="R-US_" device="R0805" value="10"/>
+<part name="R4" library="rcl" deviceset="R-US_" device="R0805" value="10"/>
+<part name="R5" library="rcl" deviceset="R-US_" device="R0805" value="10"/>
+<part name="R6" library="rcl" deviceset="R-US_" device="R0805" value="10"/>
 <part name="T1" library="zetex" deviceset="NMOSSOT23" device=""/>
 <part name="T2" library="zetex" deviceset="NMOSSOT23" device=""/>
 <part name="T3" library="zetex" deviceset="NMOSSOT23" device=""/>
 <part name="T4" library="zetex" deviceset="NMOSSOT23" device=""/>
-<part name="R7" library="rcl" deviceset="R-US_" device="R0805"/>
-<part name="R8" library="rcl" deviceset="R-US_" device="R0805"/>
-<part name="R9" library="rcl" deviceset="R-US_" device="R0805"/>
-<part name="R10" library="rcl" deviceset="R-US_" device="R0805"/>
+<part name="R7" library="rcl" deviceset="R-US_" device="R0805" value="10K"/>
+<part name="R8" library="rcl" deviceset="R-US_" device="R0805" value="10K"/>
+<part name="R9" library="rcl" deviceset="R-US_" device="R0805" value="10K"/>
+<part name="R10" library="rcl" deviceset="R-US_" device="R0805" value="10K"/>
 <part name="GND8" library="supply1" deviceset="GND" device=""/>
 <part name="GND9" library="supply1" deviceset="GND" device=""/>
@@
 </segment>
 </net>
+<net name="N$12" class="0">
+<segment>
+<pinref part="U$1" gate="G$1" pin="INT"/>
+<wire x1="50.8" y1="0" x2="63.5" y2="0" width="0.1524" layer="91"/>
+</segment>
+</net>

Commit message: Esquematico Final
Parts:
- added U$3, U$4, U$5, U$6: 1X2, headers(.05in):1X2
Connections:
- removed net ECHO: U1.GPIO16
- removed net TRIGER: U1.GPIO14
- removed net VCC_BAT: C1.1, U$2.EN, U$2.VIN
- new net N$14: T2.D, U$4.1
- new net N$16: T1.D, U$3.1
- new net N$9: T3.D, U$5.1
- new net V+: C1.1, R11.2, U$2.EN, U$2.VIN, U$3.2, U$4.2, U$5.2, U$6.2, X1-1.S
- net GND: now also C8.2, C9.2
- net N$13: now also T4.D, U$6.1; no longer IC1.SDO
- net N$7: now also IC1.SDO
- net PWM1: now also U1.SCLK; no longer U1.GPIO4
- net PWM2: now also U1.CS0; no longer U1.GPIO2
- net PWM3: now also U1.GPIO16; no longer U1.GPIO15
- net VCC: no longer R11.2, T1.D, T2.D, T3.D, T4.D, X1-1.S
Other:
- moved on the sheet: C7, C8, C9, R1, R17, R18, U1

Commit message: Esquematico Final
Connections:
- net BOOT: now also R2.2
- net GND: now also U1.GPIO15; no longer R2.1
- net VCC: now also R2.1, U1.GPIO2
Other:
- moved on the sheet: R2
Changed lines of the file:
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@@
 <part name="GND1" library="supply1" deviceset="GND" device=""/>
 <part name="R2" library="rcl" deviceset="R-US_" device="R0805"/>
-<part name="GND2" library="supply1" deviceset="GND" device=""/>
 <part name="SV1" library="con-lstb" deviceset="MA04-1" device=""/>
 <part name="GND3" library="supply1" deviceset="GND" device=""/>
@@
 <part name="SUPPLY6" library="supply2" deviceset="V+" device=""/>
 <part name="SUPPLY7" library="supply2" deviceset="V+" device=""/>
+<part name="P+3" library="supply1" deviceset="VCC" device=""/>
+<part name="P+4" library="supply1" deviceset="VCC" device=""/>
 </parts>
 <sheets>
@@
 <instance part="P+1" gate="VCC" x="15.24" y="104.14"/>
 <instance part="GND1" gate="1" x="60.96" y="63.5"/>
-<instance part="R2" gate="G$1" x="83.82" y="127" rot="R90"/>
-<instance part="GND2" gate="1" x="83.82" y="116.84"/>
+<instance part="R2" gate="G$1" x="83.82" y="137.16" rot="R270"/>
 <instance part="SV1" gate="1" x="66.04" y="134.62"/>
 <instance part="GND3" gate="1" x="76.2" y="127"/>
@@
 <instance part="SUPPLY6" gate="1" x="106.68" y="68.58"/>
 <instance part="SUPPLY7" gate="1" x="149.86" y="66.04"/>
+<instance part="P+3" gate="VCC" x="68.58" y="76.2"/>
+<instance part="P+4" gate="VCC" x="83.82" y="144.78"/>
 </instances>
 <busses>
@@
 <junction x="15.24" y="68.58"/>
 </segment>
+<segment>
+<pinref part="U1" gate="G$1" pin="GPIO2"/>
+<wire x1="55.88" y1="73.66" x2="68.58" y2="73.66" width="0.1524" layer="91"/>
+<pinref part="P+3" gate="VCC" pin="VCC"/>
+</segment>
+<segment>
+<pinref part="R2" gate="G$1" pin="1"/>
+<pinref part="P+4" gate="VCC" pin="VCC"/>
+</segment>
 </net>
 <net name="ADC" class="0">
@@
 <wire x1="73.66" y1="132.08" x2="83.82" y2="132.08" width="0.1524" layer="91"/>
 <label x="76.2" y="132.08" size="1.778" layer="95"/>
+<pinref part="R2" gate="G$1" pin="2"/>
 </segment>
 </net>
@@
 <wire x1="60.96" y1="68.58" x2="60.96" y2="66.04" width="0.1524" layer="91"/>
 <pinref part="GND1" gate="1" pin="GND"/>
-</segment>
-<segment>
-<pinref part="R2" gate="G$1" pin="1"/>
-<wire x1="83.82" y1="121.92" x2="83.82" y2="119.38" width="0.1524" layer="91"/>
-<pinref part="GND2" gate="1" pin="GND"/>
-</segment>
-<segment>
+<pinref part="U1" gate="G$1" pin="GPIO15"/>
+<wire x1="55.88" y1="71.12" x2="60.96" y2="71.12" width="0.1524" layer="91"/>
+<wire x1="60.96" y1="71.12" x2="60.96" y2="68.58" width="0.1524" layer="91"/>
+</segment>
+<segment>
