File: PCB/DIY-PCB_EAGLE/Esquematico_PCB_DIY_V1.sch (EAGLE design)
At the start: 2 parts

Commit message: Alimentacion Conmutada
Altium Version
Parts:
- added R2, R3, R4, R5, R6, R7, R8, R9: (no value), rcl:R-US_R0805
- added U$1, U$2, U$3, U$4: N-CHANNEL-MOSFET-BSS138, GeekAmmo:N-CHANNEL-MOSFET-BSS138
- added U$5: MPU-6050, invensense:MPU-6050
Connections:
- new net N$2: R2.1, U$1.G
- new net N$4: R4.1, U$2.G
- new net N$6: R6.1, U$3.G
- new net N$8: R8.1, U$4.G
- new net PWM0_MOTOR: U$1.D
- new net PWM1_MOTOR: U$2.D
- new net PWM2_MOTOR: U$3.D
- new net PWM3_MOTOR: U$4.D
- net GND: now also R3.2, R5.2, R7.2, R9.2, U$1.S, U$2.S, U$3.S, U$4.S, U$5.AD0, U$5.GND
- net I2C_SCL: now also U$5.SCL
- net I2C_SDA: now also U$5.SDA
- net PWM0: now also R2.2, R3.1
- net PWM1: now also R4.2, R5.1
- net PWM2: now also R6.2, R7.1
- net PWM3: now also R8.2, R9.1
- net VCC: now also U$5.VDD, U$5.VLOGIC
Other:
- moved on the sheet: R1, U1
