File: PCB/DIY-PCB_EAGLE/Esquematico_PCB_DIY_V1.brd (EAGLE design)
At the start: 100 x 80 mm, 2 parts

Commit message: Esquematico
Parts:
- added R2, R3, R4, R5, R6: (no value), rcl:R0805
- added SV1: (no value), con-lstb:MA04-1
- added T1, T2, T3, T4: (no value), zetex:SOT-23
Connections:
- new net N$2: R3.2, T1.3
- new net N$4: R4.2, T2.3
- new net N$5: R5.2, T3.3
- new net N$6: R6.2, T4.3
- net BOOT: now also R2.2, SV1.2
- net GND: now also R2.1, SV1.1, T1.2, T2.2, T3.2, T4.2
- net PWM0: now also R3.1
- net PWM1: now also R4.1
- net PWM2: now also R5.1
- net PWM3: now also R6.1
- net RX: now also SV1.3
- net TX: now also SV1.4
- net VCC: now also T1.1, T2.1, T3.1, T4.1
Changed lines of the file:
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@@
 <?xml version="1.0" encoding="utf-8"?>
 <!DOCTYPE eagle SYSTEM "eagle.dtd">
-<eagle version="7.5.0">
+<eagle version="7.6.0">
 <drawing>
 <settings>
@@
 <element name="R1" library="rcl" package="R0805" value="" x="6.35" y="76.2"/>
 <element name="U1" library="esp8266modules" package="ESP12E-SMD" value="" x="20.32" y="72.39"/>
+<element name="R2" library="rcl" package="R0805" value="" x="2.54" y="-3.81"/>
+<element name="SV1" library="con-lstb" package="MA04-1" value="" x="7.62" y="-8.89">
+<attribute name="OC_NEWARK" value="unknown" x="7.62" y="-8.89" size="1.778" layer="27" display="off"/>
+<attribute name="MPN" value="" x="7.62" y="-8.89" size="1.778" layer="27" display="off"/>
+<attribute name="MF" value="" x="7.62" y="-8.89" size="1.778" layer="27" display="off"/>
+<attribute name="OC_FARNELL" value="unknown" x="7.62" y="-8.89" size="1.778" layer="27" display="off"/>
+</element>
+<element name="R3" library="rcl" package="R0805" value="" x="2.54" y="-39.37"/>
+<element name="R4" library="rcl" package="R0805" value="" x="2.54" y="-44.45"/>
+<element name="R5" library="rcl" package="R0805" value="" x="2.54" y="-49.53"/>
+<element name="R6" library="rcl" package="R0805" value="" x="2.54" y="-54.61"/>
+<element name="T1" library="zetex" package="SOT-23" value="" x="2.54" y="-60.96">
+<attribute name="OC_NEWARK" value="unknown" x="2.54" y="-60.96" size="1.778" layer="27" display="off"/>
+<attribute name="MPN" value="" x="2.54" y="-60.96" size="1.778" layer="27" display="off"/>
+<attribute name="MF" value="" x="2.54" y="-60.96" size="1.778" layer="27" display="off"/>
+<attribute name="OC_FARNELL" value="unknown" x="2.54" y="-60.96" size="1.778" layer="27" display="off"/>
+</element>
+<element name="T2" library="zetex" package="SOT-23" value="" x="2.54" y="-68.58">
+<attribute name="OC_NEWARK" value="unknown" x="2.54" y="-68.58" size="1.778" layer="27" display="off"/>
+<attribute name="MPN" value="" x="2.54" y="-68.58" size="1.778" layer="27" display="off"/>
+<attribute name="MF" value="" x="2.54" y="-68.58" size="1.778" layer="27" display="off"/>
+<attribute name="OC_FARNELL" value="unknown" x="2.54" y="-68.58" size="1.778" layer="27" display="off"/>
+</element>
+<element name="T3" library="zetex" package="SOT-23" value="" x="2.54" y="-76.2">
+<attribute name="OC_NEWARK" value="unknown" x="2.54" y="-76.2" size="1.778" layer="27" display="off"/>
+<attribute name="MPN" value="" x="2.54" y="-76.2" size="1.778" layer="27" display="off"/>
+<attribute name="MF" value="" x="2.54" y="-76.2" size="1.778" layer="27" display="off"/>
+<attribute name="OC_FARNELL" value="unknown" x="2.54" y="-76.2" size="1.778" layer="27" display="off"/>
+</element>
+<element name="T4" library="zetex" package="SOT-23" value="" x="2.54" y="-83.82">
+<attribute name="OC_NEWARK" value="unknown" x="2.54" y="-83.82" size="1.778" layer="27" display="off"/>
+<attribute name="MPN" value="" x="2.54" y="-83.82" size="1.778" layer="27" display="off"/>
+<attribute name="MF" value="" x="2.54" y="-83.82" size="1.778" layer="27" display="off"/>
+<attribute name="OC_FARNELL" value="unknown" x="2.54" y="-83.82" size="1.778" layer="27" display="off"/>
+</element>
 </elements>
 <signals>
@@
 <contactref element="R1" pad="2"/>
 <contactref element="U1" pad="VCC"/>
-<wire x1="7.3" y1="76.2" x2="12.02" y2="64.19" width="0" layer="19" extent="1-1"/>
+<contactref element="T1" pad="1"/>
+<contactref element="T2" pad="1"/>
+<contactref element="T3" pad="1"/>
+<contactref element="T4" pad="1"/>
+<wire x1="12.02" y1="64.19" x2="7.3" y2="76.2" width="0" layer="19" extent="1-1"/>
+<wire x1="2.5654" y1="-61.976" x2="12.02" y2="64.19" width="0" layer="19" extent="1-1"/>
+<wire x1="2.5654" y1="-69.596" x2="2.5654" y2="-61.976" width="0" layer="19" extent="1-1"/>
+<wire x1="2.5654" y1="-77.216" x2="2.5654" y2="-69.596" width="0" layer="19" extent="1-1"/>
+<wire x1="2.5654" y1="-84.836" x2="2.5654" y2="-77.216" width="0" layer="19" extent="1-1"/>
 </signal>
 <signal name="ADC">
@@
 <signal name="TX">
 <contactref element="U1" pad="TXD0"/>
+<contactref element="SV1" pad="4"/>
+<wire x1="11.43" y1="-8.89" x2="28.42" y2="78.19" width="0" layer="19" extent="1-1"/>
 </signal>
 <signal name="RX">
 <contactref element="U1" pad="RXD0"/>
+<contactref element="SV1" pad="3"/>
+<wire x1="8.89" y1="-8.89" x2="28.42" y2="76.19" width="0" layer="19" extent="1-1"/>
 </signal>
 <signal name="PWM0">
 <contactref element="U1" pad="GPIO5"/>
+<contactref element="R3" pad="1"/>
+<wire x1="1.59" y1="-39.37" x2="28.42" y2="74.19" width="0" layer="19" extent="1-1"/>
 </signal>
 <signal name="PWM1">
 <contactref element="U1" pad="GPIO4"/>
+<contactref element="R4" pad="1"/>
+<wire x1="1.59" y1="-44.45" x2="28.42" y2="72.19" width="0" layer="19" extent="1-1"/>
 </signal>
 <signal name="BOOT">
 <contactref element="U1" pad="GPIO0"/>
+<contactref element="R2" pad="2"/>
+<contactref element="SV1" pad="2"/>
+<wire x1="3.49" y1="-3.81" x2="28.42" y2="70.19" width="0" layer="19" extent="1-1"/>
+<wire x1="6.35" y1="-8.89" x2="3.49" y2="-3.81" width="0" layer="19" extent="1-1"/>
 </signal>
 <signal name="PWM2">
 <contactref element="U1" pad="GPIO2"/>
+<contactref element="R5" pad="1"/>
+<wire x1="1.59" y1="-49.53" x2="28.42" y2="68.19" width="0" layer="19" extent="1-1"/>
 </signal>
 <signal name="PWM3">
 <contactref element="U1" pad="GPIO15"/>
+<contactref element="R6" pad="1"/>
+<wire x1="1.59" y1="-54.61" x2="28.42" y2="66.19" width="0" layer="19" extent="1-1"/>
 </signal>
 <signal name="GND">
 <contactref element="U1" pad="GND"/>
+<contactref element="R2" pad="1"/>
+<contactref element="SV1" pad="1"/>
+<contactref element="T1" pad="2"/>
+<contactref element="T2" pad="2"/>
+<contactref element="T3" pad="2"/>
+<contactref element="T4" pad="2"/>
+<wire x1="1.59" y1="-3.81" x2="28.42" y2="64.19" width="0" layer="19" extent="1-1"/>
+<wire x1="3.81" y1="-8.89" x2="1.59" y2="-3.81" width="0" layer="19" extent="1-1"/>
+<wire x1="1.6002" y1="-59.944" x2="3.81" y2="-8.89" width="0" layer="19" extent="1-1"/>
+<wire x1="1.6002" y1="-67.564" x2="1.6002" y2="-59.944" width="0" layer="19" extent="1-1"/>
+<wire x1="1.6002" y1="-75.184" x2="1.6002" y2="-67.564" width="0" layer="19" extent="1-1"/>
+<wire x1="1.6002" y1="-82.804" x2="1.6002" y2="-75.184" width="0" layer="19" extent="1-1"/>
+</signal>
+<signal name="N$2">
+<contactref element="R3" pad="2"/>
+<contactref element="T1" pad="3"/>
+<wire x1="3.49" y1="-39.37" x2="3.5306" y2="-59.944" width="0" layer="19" extent="1-1"/>
+</signal>
+<signal name="N$4">
+<contactref element="R4" pad="2"/>
+<contactref element="T2" pad="3"/>
+<wire x1="3.49" y1="-44.45" x2="3.5306" y2="-67.564" width="0" layer="19" extent="1-1"/>
+</signal>
+<signal name="N$5">
+<contactref element="R5" pad="2"/>
+<contactref element="T3" pad="3"/>
+<wire x1="3.49" y1="-49.53" x2="3.5306" y2="-75.184" width="0" layer="19" extent="1-1"/>
+</signal>
+<signal name="N$6">
+<contactref element="R6" pad="2"/>
+<contactref element="T4" pad="3"/>
+<wire x1="3.49" y1="-54.61" x2="3.5306" y2="-82.804" width="0" layer="19" extent="1-1"/>
 </signal>
 </signals>

Commit message: Esquematico Final
Parts:
- added C1: 4u7, rcl:C0805K
- added C10, C3, C6, C7: 0.1uF, rcl:C0805K
- added C11, C5, C8: 10nF, rcl:C0805K
- added C2, C9: 47uF, rcl:C0805K
- added C4: 2.2nF, rcl:C0805K
- added IC1: BMP280, bosch-bmp280:BMP280
- added L1: 4u7, inductor-neosid:MS85
- added R10, R11, R12, R7, R8, R9: 10K, rcl:R0805
- added R13, R14, R15, R16: (no value), rcl:R0805
- added R17, R18: 1K, rcl:R0805
- added U$1: MPU-6050, invensense:QFN.24.4X4
- added U$2: LM3671, texas-custom:SOT23-5
- added U$3, U$4, U$5, U$6: 1X2, headers(.05in):1X2
- added X1: 22-23-2021, con-molex:22-23-2021
- R1: value (none) -> 10K
- R3, R4, R5, R6: value (none) -> 10
- moved T4 141.4 mm to (22.4, 56.2), flipped to the bottom, turned to 270 degrees
- moved T3 122.8 mm to (19.6, 45.4), flipped to the bottom
- moved T1 122.3 mm to (31.2, 57.9), flipped to the bottom, turned to 270 degrees
- moved T2 118.5 mm to (34.8, 45.5), flipped to the bottom
- moved R6 109.4 mm to (22.5, 53.0), flipped to the bottom
- moved R3 98.8 mm to (31.2, 55.1), flipped to the bottom
- moved R5 96.0 mm to (16.2, 45.5), flipped to the bottom, turned to 90 degrees
- moved R4 94.6 mm to (32.1, 45.5), flipped to the bottom, turned to 90 degrees
- moved R2 73.7 mm to (-40.6, 55.9)
- moved SV1 67.4 mm to (38.1, 51.2), turned to 90 degrees
- moved R1 25.2 mm to (15.5, 52.7), turned to 270 degrees
- moved U1 21.3 mm to (26.7, 52.1)
Connections:
- removed net ECHO: U1.GPIO16
- removed net TRIGER: U1.GPIO14
- new net N$10: C3.1, U$1.10
- new net N$11: C4.1, U$1.20
- new net N$12: U$1.12
- new net N$13: T4.1, U$6.1
- new net N$14: T2.1, U$4.1
- new net N$16: T1.1, U$3.1
- new net N$3: L1.1, U$2.5
- new net N$7: IC1.5, R13.2, R14.1
- new net N$8: R15.1, R16.2, U$1.9
- new net N$9: T3.1, U$5.1
- new net V+: C1.1, R11.2, U$2.1, U$2.3, U$3.2, U$4.2, U$5.2, U$6.2, X1.1
- net ADC: now also R11.1, R12.1
- net BOOT: no longer R2.2
- net GND: now also C1.2, C10.2, C11.2, C2.2, C3.2, C4.2, C5.2, C6.2, C7.2, C8.2, C9.2, IC1.1, IC1.7, R10.1, R12.2, R13.1, R16.1, R7.1, R8.1, R9.1, U$1.18, U$2.2, X1.2
- net I2C_SCL: now also IC1.4, R18.1, U$1.23
- net I2C_SDA: now also IC1.3, R17.1, U$1.24
- net PWM0: now also R7.2
- net PWM1: now also R8.2, U1.SCLK; no longer U1.GPIO4
- net PWM2: now also R10.2, U1.CS0; no longer U1.GPIO2
- net PWM3: now also R9.2, U1.GPIO16; no longer U1.GPIO15
- net VCC: now also C10.1, C11.1, C2.1, C5.1, C6.1, C7.1, C8.1, C9.1, IC1.2, IC1.6, IC1.8, L1.2, R14.2, R15.2, R17.2, R18.2, U$1.13, U$1.8, U$2.4; no longer T1.1, T2.1, T3.1, T4.1
Routing:
- net GND: track 0.00 -> 36.4 mm
- net I2C_SDA: track 0.00 -> 15.6 mm
- net I2C_SCL: track 0.00 -> 13.4 mm
- net N$13: track 0.00 -> 10.2 mm
- net PWM1: track 0.00 -> 6.31 mm
- net N$16: track 0.00 -> 5.71 mm
- net N$9: track 0.00 -> 5.66 mm
- net PWM0: track 0.00 -> 4.78 mm
- net N$5: track 0.00 -> 2.47 mm
- net PWM2: track 0.00 -> 2.38 mm
- net N$6: track 0.00 -> 2.29 mm
- net PWM3: track 0.00 -> 2.22 mm
- net N$2: track 0.00 -> 1.82 mm
- net N$4: track 0.00 -> 1.77 mm

Commit message: Esquematico Final
Connections:
- net BOOT: now also R2.2
- net GND: now also U1.GPIO15; no longer R2.1
- net VCC: now also R2.1, U1.GPIO2
Changed lines of the file:
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@@
 <contactref element="C8" pad="1"/>
 <contactref element="C9" pad="1"/>
+<contactref element="U1" pad="GPIO2"/>
+<contactref element="R2" pad="1"/>
+<wire x1="33.671" y1="39.116" x2="34.77" y2="47.87" width="0" layer="19" extent="1-1"/>
 <wire x1="32.8629" y1="37.145" x2="33.671" y2="39.116" width="0" layer="19" extent="1-1"/>
 <wire x1="28.321" y1="38.689" x2="32.8629" y2="37.145" width="0" layer="19" extent="1-1"/>
@@
 <wire x1="-37.83" y1="52.07" x2="-32.75" y2="52.07" width="0" layer="19" extent="1-1"/>
 <wire x1="-42.91" y1="52.07" x2="-37.83" y2="52.07" width="0" layer="19" extent="1-1"/>
+<wire x1="-41.59" y1="55.88" x2="-42.91" y2="52.07" width="0" layer="19" extent="1-1"/>
 <wire x1="-47.99" y1="52.07" x2="-42.91" y2="52.07" width="0" layer="19" extent="1-1"/>
 <wire x1="-51.8" y1="46.99" x2="-47.99" y2="52.07" width="0" layer="19" extent="1-1"/>
@@
 <contactref element="U1" pad="GPIO0"/>
 <contactref element="SV1" pad="2"/>
+<contactref element="R2" pad="2"/>
 <wire x1="34.77" y1="49.87" x2="38.1" y2="49.911" width="0" layer="19" extent="1-1"/>
+<wire x1="-39.69" y1="55.88" x2="34.77" y2="49.87" width="0" layer="19" extent="1-1"/>
 </signal>
 <signal name="PWM2">
@@
 <signal name="GND">
 <contactref element="U1" pad="GND"/>
-<contactref element="R2" pad="1"/>
 <contactref element="SV1" pad="1"/>
 <contactref element="T1" pad="2"/>
@@
 <wire x1="30.875" y1="48.3" x2="34.6506" y2="48.3" width="0.5" layer="16"/>
 <wire x1="34.6506" y1="48.3" x2="35.7378" y2="47.2128" width="0.5" layer="16"/>
-<wire x1="30.875" y1="48.3" x2="30.292" y2="52.959" width="0" layer="19" extent="16-16"/>
-<wire x1="34.77" y1="43.87" x2="35.7378" y2="46.482" width="0" layer="19" extent="1-16"/>
-<wire x1="35.671" y1="39.116" x2="34.77" y2="43.87" width="0" layer="19" extent="1-1"/>
-<wire x1="37.592" y1="39.354" x2="35.671" y2="39.116" width="0" layer="19" extent="1-1"/>
-<wire x1="35.4631" y1="36.195" x2="35.671" y2="39.116" width="0" layer="19" extent="1-1"/>
-<wire x1="38.608" y1="32.385" x2="35.4631" y2="36.195" width="0" layer="19" extent="1-1"/>
-<wire x1="21.477" y1="50.783" x2="30.292" y2="52.959" width="0" layer="19" extent="16-16"/>
-<wire x1="13.808" y1="46.451" x2="21.477" y2="50.783" width="0" layer="19" extent="16-16"/>
-<wire x1="14.271" y1="36.953" x2="20.5418" y2="46.461" width="0" layer="19" extent="1-16"/>
-<wire x1="14.921" y1="35.353" x2="14.271" y2="36.953" width="0" layer="19" extent="1-1"/>
-<wire x1="23.438" y1="37.699" x2="14.921" y2="35.353" width="0" layer="19" extent="1-1"/>
-<wire x1="20.14" y1="32.185" x2="23.438" y2="37.699" width="0" layer="19" extent="1-1"/>
-<wire x1="-15.51" y1="52.07" x2="14.271" y2="36.953" width="0" layer="19" extent="1-1"/>
-<wire x1="-17.46" y1="55.88" x2="-15.51" y2="52.07" width="0" layer="19" extent="1-1"/>
-<wire x1="-20.59" y1="52.07" x2="-17.46" y2="55.88" width="0" layer="19" extent="1-1"/>
-<wire x1="-30.75" y1="52.07" x2="-20.59" y2="52.07" width="0" layer="19" extent="1-1"/>
-<wire x1="-35.83" y1="52.07" x2="-30.75" y2="52.07" width="0" layer="19" extent="1-1"/>
-<wire x1="-36.51" y1="55.88" x2="-35.83" y2="52.07" width="0" layer="19" extent="1-1"/>
-<wire x1="-41.59" y1="55.88" x2="-36.51" y2="55.88" width="0" layer="19" extent="1-1"/>
-<wire x1="-40.91" y1="52.07" x2="-41.59" y2="55.88" width="0" layer="19" extent="1-1"/>
-<wire x1="-45.99" y1="52.07" x2="-40.91" y2="52.07" width="0" layer="19" extent="1-1"/>
-<wire x1="-44.72" y1="46.99" x2="-45.99" y2="52.07" width="0" layer="19" extent="1-1"/>
-<wire x1="-49.8" y1="46.99" x2="-44.72" y2="46.99" width="0" layer="19" extent="1-1"/>
-<wire x1="-39.69" y1="33.02" x2="-44.72" y2="46.99" width="0" layer="19" extent="1-1"/>
 <wire x1="21.363" y1="57.1538" x2="20.7288" y2="57.1538" width="0.5" layer="16"/>
 <wire x1="20.7288" y1="57.1538" x2="20.075" y2="56.5" width="0.5" layer="16"/>
@@
 <wire x1="13.875" y1="47.625" x2="13.875" y2="46.518" width="0.5" layer="16"/>
 <wire x1="13.875" y1="46.518" x2="13.808" y2="46.451" width="0.5" layer="16"/>
+<contactref element="U1" pad="GPIO15"/>
+<wire x1="30.875" y1="48.3" x2="30.233" y2="52.9" width="0" layer="19" extent="16-16"/>
+<wire x1="34.77" y1="45.87" x2="35.7378" y2="46.482" width="0" layer="19" extent="1-16"/>
+<wire x1="34.77" y1="43.87" x2="34.77" y2="45.87" width="0" layer="19" extent="1-1"/>
+<wire x1="35.671" y1="39.116" x2="34.77" y2="43.87" width="0" layer="19" extent="1-1"/>
+<wire x1="37.592" y1="39.354" x2="35.671" y2="39.116" width="0" layer="19" extent="1-1"/>
+<wire x1="35.4631" y1="36.195" x2="35.671" y2="39.116" width="0" layer="19" extent="1-1"/>
+<wire x1="38.608" y1="32.385" x2="35.4631" y2="36.195" width="0" layer="19" extent="1-1"/>
+<wire x1="21.363" y1="57.1538" x2="28.95" y2="58.525" width="0" layer="19" extent="16-16"/>
+<wire x1="20.1" y1="48" x2="20.675" y2="50.925" width="0" layer="19" extent="16-16"/>
+<wire x1="23.438" y1="37.699" x2="20.5418" y2="46.461" width="0" layer="19" extent="1-16"/>
+<wire x1="20.14" y1="32.185" x2="23.438" y2="37.699" width="0" layer="19" extent="1-1"/>
+<wire x1="14.921" y1="35.353" x2="20.14" y2="32.185" width="0" layer="19" extent="1-1"/>
+<wire x1="14.271" y1="36.953" x2="14.921" y2="35.353" width="0" layer="19" extent="1-1"/>
+<wire x1="-15.51" y1="52.07" x2="13.875" y2="47.625" width="0" layer="19" extent="1-16"/>
+<wire x1="-17.46" y1="55.88" x2="-15.51" y2="52.07" width="0" layer="19" extent="1-1"/>
+<wire x1="-20.59" y1="52.07" x2="-17.46" y2="55.88" width="0" layer="19" extent="1-1"/>
+<wire x1="-30.75" y1="52.07" x2="-20.59" y2="52.07" width="0" layer="19" extent="1-1"/>
+<wire x1="-35.83" y1="52.07" x2="-30.75" y2="52.07" width="0" layer="19" extent="1-1"/>
+<wire x1="-36.51" y1="55.88" x2="-35.83" y2="52.07" width="0" layer="19" extent="1-1"/>
+<wire x1="-40.91" y1="52.07" x2="-35.83" y2="52.07" width="0" layer="19" extent="1-1"/>
+<wire x1="-45.99" y1="52.07" x2="-40.91" y2="52.07" width="0" layer="19" extent="1-1"/>
+<wire x1="-44.72" y1="46.99" x2="-45.99" y2="52.07" width="0" layer="19" extent="1-1"/>
+<wire x1="-49.8" y1="46.99" x2="-44.72" y2="46.99" width="0" layer="19" extent="1-1"/>
+<wire x1="-39.69" y1="33.02" x2="-44.72" y2="46.99" width="0" layer="19" extent="1-1"/>
 </signal>
 <signal name="N$2">
